File: KiCAD_Proj (MCU datalogger).kicad_sch (KiCad schematic)
At the start: 25 parts, among them U1 24LC1025-I_SM, U2 DS1337S_, U3 24LC1025-I_SM, U4 ATMEGA328P-AU, Y1 32.768 KHz, Y2 16MHz

Commit message: Compeleted the page settings.
Other:
- removed sheet Connectors
- added sheet Untitled Sheet (C:/Project Punk/KiCAD Proj/KiCAD_Proj (MCU datalogger [2 layer])/Connectors.kicad_sch/Connectors.kicad_sch)
- company: (none) -> MCU Datalogger
Changed lines of the file:
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@@
 	(generator_version "9.0")
 	(paper "A4")
+	(title_block
+		(date "916/2025")
+		(company "MCU Datalogger")
+		(comment 1 "LAUDE, RUSELLE RAE D.")
+		(comment 2 "BSECE - 1C")
+		(comment 3 "ELECTRONICS ENGINEERING DEPARTMENT")
+		(comment 4 "COLLEGE OF ENGINEERING")
+		(comment 5 "TECHNOLOGICAL UNIVERSITY OF THE PHILIPPINES")
+	)
 	(text "EEPROM"
 		(exclude_from_sim no)
@@
 	(wire
 		(pts
-			(xy 172.72 125.73) (xy 165.1 125.73)
-		)
-		(stroke
-			(width 0)
-			(type default)
-		)
-	)
-	(wire
-		(pts
 			(xy 91.44 152.4) (xy 104.14 152.4)
 		)
@@
 	(wire
 		(pts
-			(xy 165.1 125.73) (xy 165.1 127)
+			(xy 153.67 123.19) (xy 161.29 123.19)
+		)
+		(stroke
+			(width 0)
+			(type default)
+		)
+	)
+	(wire
+		(pts
+			(xy 153.67 125.73) (xy 153.67 127)
 		)
 		(stroke
@@
 	(wire
 		(pts
+			(xy 153.67 125.73) (xy 161.29 125.73)
+		)
+		(stroke
+			(width 0)
+			(type default)
+		)
+	)
+	(wire
+		(pts
 			(xy 156.21 48.26) (xy 167.64 48.26)
 		)
@@
 	(wire
 		(pts
-			(xy 165.1 123.19) (xy 172.72 123.19)
-		)
-		(stroke
-			(width 0)
-			(type default)
-		)
-	)
-	(wire
-		(pts
 			(xy 241.3 95.25) (xy 241.3 97.79)
 		)
@@
 	)
 	(label "RESET"
-		(at 172.72 149.86 180)
+		(at 161.29 149.86 180)
 		(effects
 			(font
@@
 	)
 	(label "RX"
-		(at 172.72 140.97 180)
+		(at 161.29 140.97 180)
 		(effects
 			(font
@@
 	)
 	(label "D4"
-		(at 196.85 134.62 0)
+		(at 185.42 134.62 0)
 		(effects
 			(font
@@
 	)
 	(label "SCK"
-		(at 172.72 133.35 180)
+		(at 161.29 133.35 180)
 		(effects
 			(font
@@
 	)
 	(label "MOSI"
-		(at 172.72 144.78 180)
+		(at 161.29 144.78 180)
 		(effects
 			(font
@@
 	)
 	(label "D2"
-		(at 196.85 129.54 0)
+		(at 185.42 129.54 0)
 		(effects
 			(font
@@
 	)
 	(label "SDA"
-		(at 172.72 130.81 180)
+		(at 161.29 130.81 180)
 		(effects
 			(font
@@
 	)
 	(label "D5"
-		(at 196.85 137.16 0)
+		(at 185.42 137.16 0)
 		(effects
 			(font
@@
 	)
 	(label "D6"
-		(at 196.85 139.7 0)
+		(at 185.42 139.7 0)
 		(effects
 			(font
@@
 	)
 	(label "D7"
-		(at 196.85 142.24 0)
+		(at 185.42 142.24 0)
 		(effects
 			(font
@@
 	)
 	(label "D8"
-		(at 196.85 144.78 0)
+		(at 185.42 144.78 0)
 		(effects
 			(font
@@
 	)
 	(label "MISO"
-		(at 172.72 147.32 180)
+		(at 161.29 147.32 180)
 		(effects
 			(font
@@
 	)
 	(label "TX"
-		(at 172.72 138.43 180)
+		(at 161.29 138.43 180)
 		(effects
 			(font
@@
 	)
 	(label "D3"
-		(at 196.85 132.08 0)
+		(at 185.42 132.08 0)
 		(effects
 			(font
@@
 	)
 	(label "Vcc"
-		(at 165.1 123.19 180)
+		(at 153.67 123.19 180)
 		(effects
 			(font
@@
 	(symbol
 		(lib_id "power:GND")
-		(at 165.1 127 0)
+		(at 153.67 127 0)
 		(unit 1)
 		(exclude_from_sim no)
@@
 		(fields_autoplaced yes)
 		(property "Reference" "#PWR03"
-			(at 165.1 133.35 0)
+			(at 153.67 133.35 0)
 			(effects
 				(font
@@
 		)
 		(property "Value" "GND"
-			(at 165.1 132.08 0)
+			(at 153.67 132.08 0)
 			(effects
 				(font
@@
 		)
 		(property "Footprint" ""
-			(at 165.1 127 0)
+			(at 153.67 127 0)
 			(effects
 				(font
@@
 		)
 		(property "Datasheet" ""
-			(at 165.1 127 0)
+			(at 153.67 127 0)
 			(effects
 				(font
@@
 		)
 		(property "Description" "Power symbol creates a global label with name \"GND\" , ground"
-			(at 165.1 127 0)
+			(at 153.67 127 0)
 			(effects
 				(font
@@
 	)
 	(sheet
-		(at 172.72 120.65)
+		(at 161.29 120.65)
 		(size 24.13 31.75)
 		(exclude_from_sim no)
@@
 			(color 0 0 0 0.0000)
 		)
-		(property "Sheetname" "Connectors"
-			(at 172.72 119.9384 0)
+		(property "Sheetname" "Untitled Sheet"
+			(at 161.29 119.9384 0)
 			(effects
 				(font
@@
 			)
 		)
-		(property "Sheetfile" "C:/Project Punk/KiCAD Proj/KiCAD_Proj (MCU datalogger)/Connectors.kicad_sch/Connectors.kicad_sch"
-			(at 172.72 152.9846 0)
+		(property "Sheetfile" "C:/Project Punk/KiCAD Proj/KiCAD_Proj (MCU datalogger [2 layer])/Connectors.kicad_sch/Connectors.kicad_sch"
+			(at 161.29 152.9846 0)
 			(effects
 				(font
@@
 			)
 		)
-		(pin "Vcc" passive
-			(at 172.72 123.19 180)
+		(pin "D2" tri_state
+			(at 185.42 129.54 0)
 			(effects
 				(font
 					(size 1.27 1.27)
 				)
-				(justify left)
+				(justify right)
 			)
 		)
-		(pin "GND" passive
-			(at 172.72 125.73 180)
+		(pin "D3" tri_state
+			(at 185.42 132.08 0)
 			(effects
 				(font
 					(size 1.27 1.27)
 				)
-				(justify left)
+				(justify right)
 			)
 		)
-		(pin "SDA" tri_state
-			(at 172.72 130.81 180)
+		(pin "D4" tri_state
+			(at 185.42 134.62 0)
 			(effects
 				(font
 					(size 1.27 1.27)
 				)
-				(justify left)
+				(justify right)
 			)
 		)
-		(pin "SCK" passive
-			(at 172.72 133.35 180)
+		(pin "D5" tri_state
+			(at 185.42 137.16 0)
 			(effects
 				(font
 					(size 1.27 1.27)
 				)
-				(justify left)
+				(justify right)
 			)
 		)
-		(pin "TX" output
-			(at 172.72 138.43 180)
+		(pin "D6" tri_state
+			(at 185.42 139.7 0)
 			(effects
 				(font
 					(size 1.27 1.27)
 				)
-				(justify left)
+				(justify right)
 			)
 		)
-		(pin "RX" input
-			(at 172.72 140.97 180)
+		(pin "D7" tri_state
+			(at 185.42 142.24 0)
 			(effects
 				(font
 					(size 1.27 1.27)
 				)
-				(justify left)
+				(justify right)
 			)
 		)
-		(pin "MOSI" input
-			(at 172.72 144.78 180)
+		(pin "D8" tri_state
+			(at 185.42 144.78 0)
 			(effects
 				(font
 					(size 1.27 1.27)
 				)
-				(justify left)
+				(justify right)
 			)
 		)
-		(pin "MISO" output
-			(at 172.72 147.32 180)
+		(pin "GND" passive
+			(at 161.29 125.73 180)
 			(effects
 				(font
@@
 			)
 		)
-		(pin "RESET" passive
-			(at 172.72 149.86 180)
+		(pin "Vcc" passive
+			(at 161.29 123.19 180)
 			(effects
 				(font
@@
 			)
 		)
-		(pin "D2" tri_state
-			(at 196.85 129.54 0)
+		(pin "MISO" output
+			(at 161.29 147.32 180)
 			(effects
 				(font
 					(size 1.27 1.27)
 				)
-				(justify right)
+				(justify left)
 			)
 		)
-		(pin "D3" tri_state
-			(at 196.85 132.08 0)
+		(pin "MOSI" input
+			(at 161.29 144.78 180)
 			(effects
 				(font
 					(size 1.27 1.27)
 				)
-				(justify right)
+				(justify left)
 			)
 		)
-		(pin "D4" tri_state
-			(at 196.85 134.62 0)
+		(pin "RESET" passive
+			(at 161.29 149.86 180)
 			(effects
 				(font
 					(size 1.27 1.27)
 				)
-				(justify right)
+				(justify left)
 			)
 		)
-		(pin "D5" tri_state
-			(at 196.85 137.16 0)
+		(pin "RX" input
+			(at 161.29 140.97 180)
 			(effects
 				(font
 					(size 1.27 1.27)
 				)
-				(justify right)
+				(justify left)
 			)
 		)
-		(pin "D6" tri_state
-			(at 196.85 139.7 0)
+		(pin "SCK" passive
+			(at 161.29 133.35 180)
 			(effects
 				(font
 					(size 1.27 1.27)
 				)
-				(justify right)
+				(justify left)
 			)
 		)
-		(pin "D7" tri_state
-			(at 196.85 142.24 0)
+		(pin "SDA" tri_state
+			(at 161.29 130.81 180)
 			(effects
 				(font
 					(size 1.27 1.27)
 				)
-				(justify right)
+				(justify left)
 			)
 		)
-		(pin "D8" tri_state
-			(at 196.85 144.78 0)
+		(pin "TX" output
+			(at 161.29 138.43 180)
 			(effects
 				(font
 					(size 1.27 1.27)
 				)
-				(justify right)
+				(justify left)
 			)
 		)
@@
 			(project "KiCAD_Proj (MCU datalogger)"
 				(path "/4bd39814-648a-43e5-9d59-9775154104be"
-					(page "2")
+					(page "3")
 				)
 			)
